File: hardware/badge.brd (EAGLE design)
At the start: 162.6 x 101.6 mm, 64 parts, among them IC1 DA7280-00FVC, J7 MDT420E01001NOTECARD, J9 DX07S016JA1R1500, Q1 2.5A/30V/105mΩ, U1 RP2040, U2 W25Q512JVEIM, U3 LP3961EMP-3.3, U4 BME688, U5 BMI270, Y1 ABLS-12.000MHZ-B4-T

Commit message: hardware changes
Parts:
- removed R4: 1k, SparkFun-Resistors:0603
Connections:
- removed net !BOOT: R4.2, S1.1
- net 3.3V: no longer D2.A
- net GND: now also D2.C
- net N$7: now also D2.A; no longer D2.C
- net QSPI_CS: now also S1.1; no longer R4.1
Routing:
- net QSPI_CS: track 41.0 -> 67.1 mm, vias 0 -> 2
- net !BOOT: track 24.9 -> 0.00 mm, vias 2 -> 0
- net 3.3V: track 170.1 -> 166.9 mm, vias 23 -> 22
- net N$7: track 5.42 -> 6.91 mm
Changed lines of the file:
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@@
 </layers>
 <board>
-<fusionsync huburn="a.cGVyc29uYWw6dWUyYWE1ODAx" projecturn="a.cGVyc29uYWw6dWUyYWE1ODAxIzIwMTcxMjAyMTA2ODM1MjI2" f3durn="urn:adsk.wipprod:dm.lineage:wzztGgUqRoWfCWV1aP6Izg" pcbguid="" lastpulledtime="2022-12-31T02:41:45Z" lastsyncedchangeguid="" latestrevisionid="529266a5-a92a-4c9b-94a6-aed5478d102b" lastsyncedrevisionid="529266a5-a92a-4c9b-94a6-aed5478d102b" lastboardhashguid="" lastpushedtime="" linktopcb3d="true"/>
+<fusionsync huburn="a.cGVyc29uYWw6dWUyYWE1ODAx" projecturn="a.cGVyc29uYWw6dWUyYWE1ODAxIzIwMTcxMjAyMTA2ODM1MjI2" f3durn="urn:adsk.wipprod:dm.lineage:wzztGgUqRoWfCWV1aP6Izg" pcbguid="" lastpulledtime="2022-12-31T02:41:45Z" lastsyncedchangeguid="" latestrevisionid="529266a5-a92a-4c9b-94a6-aed5478d102b" lastsyncedrevisionid="529266a5-a92a-4c9b-94a6-aed5478d102b" lastboardhashguid="" lastpushedtime="" linktopcb3d="false"/>
 <plain>
 <wire x1="90" y1="96.198" x2="90" y2="99.198" width="0" layer="20" curve="180" locked="yes"/>
@@
 <attribute name="VALUE" x="28.0162" y="79.4512" size="0.6096" layer="27" font="vector" ratio="20" rot="R90" align="top-center"/>
 </element>
-<element name="R4" library="SparkFun-Resistors" library_urn="urn:adsk.eagle:library:532" package="0603" package3d_urn="urn:adsk.eagle:package:39650/1" value="1k" x="25.2222" y="79.4512" smashed="yes" rot="R90">
-<attribute name="NAME" x="25.2222" y="82.4992" size="1.016" layer="25" font="vector" ratio="20" rot="R180" align="bottom-center"/>
-<attribute name="PROD_ID" value="RES-07856" x="153.4922" y="117.5512" size="1.778" layer="27" rot="R90" display="off"/>
-<attribute name="VALUE" x="25.9842" y="79.4512" size="0.6096" layer="27" font="vector" ratio="20" rot="R90" align="top-center"/>
-</element>
 <element name="R5" library="SparkFun-Resistors" library_urn="urn:adsk.eagle:library:532" package="0603" package3d_urn="urn:adsk.eagle:package:39650/1" value="5.1k" x="10.8712" y="89.9922" smashed="yes" rot="R90">
 <attribute name="NAME" x="10.8712" y="88.0872" size="1.27" layer="25" font="vector" ratio="20" rot="R180" align="bottom-center"/>
@@
 <wire x1="46.7614" y1="69.342" x2="45.1817" y2="69.342" width="0.1524" layer="1"/>
 <wire x1="45.1817" y1="69.342" x2="45.0286" y2="69.4951" width="0.1524" layer="1"/>
+<contactref element="D2" pad="C"/>
 </signal>
 <signal name="VOUT">
@@
 <wire x1="144.78" y1="8.8646" x2="145.7198" y2="8.8646" width="0.1524" layer="15"/>
 <wire x1="129.8194" y1="4.9022" x2="131.191" y2="4.9022" width="0.1524" layer="15"/>
-<contactref element="D2" pad="A"/>
-<wire x1="43.5984" y1="99.0854" x2="41.656" y2="99.0854" width="0.1524" layer="1"/>
-<wire x1="41.656" y1="99.0854" x2="41.3512" y2="98.7806" width="0.1524" layer="1"/>
-<via x="41.3512" y="98.7806" extent="1-16" drill="0.35"/>
-<wire x1="41.3512" y1="98.7806" x2="41.3512" y2="97.917" width="0.1524" layer="15"/>
 </signal>
 <signal name="SWCLK">
@@
 <contactref element="U2" pad="1"/>
 <contactref element="R3" pad="1"/>
-<contactref element="R4" pad="1"/>
 <wire x1="27.2542" y1="78.6012" x2="27.178" y2="78.6012" width="0.4064" layer="1"/>
-<wire x1="27.178" y1="78.6012" x2="25.2222" y2="78.6012" width="0.4064" layer="1"/>
 <wire x1="30.9792" y1="76.0222" x2="27.7368" y2="76.0222" width="0.254" layer="1"/>
 <wire x1="27.178" y1="76.581" x2="27.178" y2="78.6012" width="0.254" layer="1"/>
@@
 <wire x1="27.0256" y1="75.311" x2="27.7368" y2="76.0222" width="0.1524" layer="1"/>
 <wire x1="41.7322" y1="79.58735" x2="42.4307" y2="78.88885" width="0.1524" layer="1"/>
-</signal>
-<signal name="!BOOT">
-<contactref element="R4" pad="2"/>
 <contactref element="S1" pad="1"/>
-<wire x1="25.2222" y1="80.3012" x2="25.2222" y2="83.312" width="0.1524" layer="1"/>
-<wire x1="25.2222" y1="83.312" x2="25.5016" y2="83.5914" width="0.1524" layer="1"/>
 <via x="25.5016" y="83.5914" extent="1-16" drill="0.381"/>
 <wire x1="25.5016" y1="83.5914" x2="25.5016" y2="94.6404" width="0.1524" layer="16"/>
@@
 <wire x1="25.781" y1="94.9198" x2="29.3624" y2="94.9198" width="0.1524" layer="16"/>
 <wire x1="29.6164" y1="95.1738" x2="29.6164" y2="97.5614" width="0.1524" layer="16"/>
+<wire x1="27.2542" y1="78.6012" x2="25.7928" y2="78.6012" width="0.254" layer="1"/>
+<wire x1="25.5016" y1="78.8924" x2="25.5016" y2="83.5914" width="0.254" layer="1"/>
+<wire x1="25.7928" y1="78.6012" x2="25.5016" y2="78.8924" width="0.254" layer="1"/>
 </signal>
 <signal name="!RESET">
@@
 <signal name="N$7">
 <contactref element="R10" pad="2"/>
-<contactref element="D2" pad="C"/>
-<wire x1="45.466" y1="93.7124" x2="45.466" y2="98.9718" width="0.1524" layer="1"/>
-<wire x1="45.466" y1="98.9718" x2="45.3524" y2="99.0854" width="0.1524" layer="1"/>
+<contactref element="D2" pad="A"/>
+<wire x1="45.466" y1="93.7124" x2="45.466" y2="95.6818" width="0.1524" layer="1"/>
+<wire x1="43.5984" y1="96.254" x2="43.5984" y2="99.0854" width="0.1524" layer="1"/>
+<wire x1="45.466" y1="95.6818" x2="45.1612" y2="95.9866" width="0.1524" layer="1"/>
+<wire x1="45.1612" y1="95.9866" x2="43.8658" y2="95.9866" width="0.1524" layer="1"/>
+<wire x1="43.8658" y1="95.9866" x2="43.5984" y2="96.254" width="0.1524" layer="1"/>
 </signal>
 </signals>
