File: hardware/badge.sch (EAGLE design)
At the start: 64 parts, among them IC1 DA7280-00FVC, J7 MDT420E01001NOTECARD, J9 DX07S016JA1R1500, Q1 2.5A/30V/105mΩ, U1 RP2040, U2 W25Q512JVEIM, U3 LP3961EMP-3.3, U4 BME688, U5 BMI270, Y1 ABLS-12.000MHZ-B4-T

Commit message: hardware changes
Parts:
- removed R4: 1k, SparkFun-Resistors:1KOHM-0603-1/10W-1%
Connections:
- removed net !BOOT: R4.2, S1.1
- net 3.3V: no longer D2.A
- net GND: now also D2.C
- net N$7: now also D2.A; no longer D2.C
- net QSPI_CS: now also S1.1; no longer R4.1
Other:
- moved on the sheet: D2
Changed lines of the file:
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@@
 <part name="S2" library="SparkFun-Switches" library_urn="urn:adsk.eagle:library:535" deviceset="MOMENTARY-SWITCH-SPST" device="-SMD-6.0X3.5MM" package3d_urn="urn:adsk.eagle:package:40165/1"/>
 <part name="R3" library="SparkFun-Resistors" library_urn="urn:adsk.eagle:library:532" deviceset="10KOHM" device="-0603-1/10W-1%" package3d_urn="urn:adsk.eagle:package:39650/1" value="10k"/>
-<part name="R4" library="SparkFun-Resistors" library_urn="urn:adsk.eagle:library:532" deviceset="1KOHM" device="-0603-1/10W-1%" package3d_urn="urn:adsk.eagle:package:39650/1" value="1k"/>
 <part name="GND6" library="SparkFun-PowerSymbols" library_urn="urn:adsk.eagle:library:530" deviceset="GND" device=""/>
 <part name="GND7" library="SparkFun-PowerSymbols" library_urn="urn:adsk.eagle:library:530" deviceset="GND" device=""/>
@@
 <part name="R10" library="SparkFun-Resistors" library_urn="urn:adsk.eagle:library:532" deviceset="330OHM" device="-0603-1/10W-1%" package3d_urn="urn:adsk.eagle:package:39650/1" value="330"/>
 <part name="D2" library="SparkFun-LED" library_urn="urn:adsk.eagle:library:529" deviceset="LED-BLUE" device="0603" package3d_urn="urn:adsk.eagle:package:39354/1" value="BLUE"/>
-<part name="SUPPLY10" library="SparkFun-PowerSymbols" library_urn="urn:adsk.eagle:library:530" deviceset="3.3V" device=""/>
 <part name="LED1" library="adafruit" library_urn="urn:adsk.eagle:library:420" deviceset="RGBLED" device="5050" package3d_urn="urn:adsk.eagle:package:6240865/1"/>
 <part name="SUPPLY11" library="SparkFun-PowerSymbols" library_urn="urn:adsk.eagle:library:530" deviceset="3.3V" device=""/>
@@
 <part name="C22" library="SparkFun-Capacitors" library_urn="urn:adsk.eagle:library:510" deviceset="0.1UF" device="-0603-25V-(+80/-20%)" package3d_urn="urn:adsk.eagle:package:37414/1" value="0.1uF"/>
 <part name="GND9" library="SparkFun-PowerSymbols" library_urn="urn:adsk.eagle:library:530" deviceset="GND" device=""/>
+<part name="GND27" library="SparkFun-PowerSymbols" library_urn="urn:adsk.eagle:library:530" deviceset="GND" device=""/>
 </parts>
 <sheets>
@@
 <attribute name="VALUE" x="215.392" y="154.178" size="1.27" layer="96" font="vector" ratio="20" align="top-center"/>
 </instance>
-<instance part="R4" gate="G$1" x="175.26" y="139.7" smashed="yes" rot="R90">
-<attribute name="NAME" x="173.736" y="144.018" size="1.27" layer="95" font="vector" ratio="20" rot="R180" align="bottom-center"/>
-<attribute name="VALUE" x="173.99" y="135.382" size="1.27" layer="96" font="vector" ratio="20" rot="R180" align="top-center"/>
-</instance>
 <instance part="GND6" gate="1" x="185.42" y="91.44" smashed="yes">
 <attribute name="VALUE" x="185.42" y="91.186" size="1.27" layer="96" font="vector" ratio="20" align="top-center"/>
@@
 <attribute name="VALUE" x="116.078" y="80.264" size="1.27" layer="96" font="vector" ratio="20" align="top-center"/>
 </instance>
-<instance part="D2" gate="G$1" x="127" y="78.74" smashed="yes" rot="R270">
-<attribute name="NAME" x="127.508" y="77.089" size="1.27" layer="95" font="vector" ratio="20"/>
-<attribute name="VALUE" x="119.888" y="78.613" size="1.27" layer="96" font="vector" ratio="20" align="top-left"/>
-</instance>
-<instance part="SUPPLY10" gate="G$1" x="137.668" y="87.122" smashed="yes">
-<attribute name="VALUE" x="137.668" y="89.916" size="1.27" layer="96" font="vector" ratio="20" align="bottom-center"/>
+<instance part="D2" gate="G$1" x="127" y="78.74" smashed="yes" rot="R90">
+<attribute name="NAME" x="126.492" y="80.391" size="1.27" layer="95" font="vector" ratio="20" rot="R180"/>
+<attribute name="VALUE" x="134.112" y="78.867" size="1.27" layer="96" font="vector" ratio="20" rot="R180" align="top-left"/>
 </instance>
 <instance part="LED1" gate="G$1" x="228.6" y="58.42" smashed="yes" rot="R180">
@@
 <attribute name="NAME" x="26.162" y="91.948" size="1.27" layer="95" font="vector" ratio="20" align="bottom-center"/>
 <attribute name="VALUE" x="34.544" y="92.964" size="1.27" layer="96" font="vector" ratio="20" align="top-center"/>
+</instance>
+<instance part="GND27" gate="1" x="139.192" y="66.548" smashed="yes">
+<attribute name="VALUE" x="139.192" y="66.294" size="1.27" layer="96" font="vector" ratio="20" align="top-center"/>
 </instance>
 </instances>
@@
 <wire x1="52.07" y1="15.24" x2="73.66" y2="15.24" width="0.1524" layer="91"/>
 <junction x="73.66" y="15.24"/>
+</segment>
+<segment>
+<pinref part="GND27" gate="1" pin="GND"/>
+<pinref part="D2" gate="G$1" pin="C"/>
+<wire x1="139.192" y1="69.088" x2="139.192" y2="78.74" width="0.1524" layer="91"/>
+<wire x1="139.192" y1="78.74" x2="132.08" y2="78.74" width="0.1524" layer="91"/>
 </segment>
 </net>
@@
 </segment>
 <segment>
-<pinref part="SUPPLY10" gate="G$1" pin="3.3V"/>
-<wire x1="137.668" y1="78.74" x2="137.668" y2="87.122" width="0.1524" layer="91"/>
-<pinref part="D2" gate="G$1" pin="A"/>
-<wire x1="129.54" y1="78.74" x2="137.668" y2="78.74" width="0.1524" layer="91"/>
-</segment>
-<segment>
 <pinref part="LED1" gate="G$1" pin="RED_A"/>
 <pinref part="SUPPLY11" gate="G$1" pin="3.3V"/>
@@
 <wire x1="185.928" y1="152.4" x2="185.928" y2="129.54" width="0.1524" layer="91"/>
 <junction x="185.928" y="129.54"/>
-<pinref part="R4" gate="G$1" pin="1"/>
-<wire x1="175.26" y1="134.62" x2="175.26" y2="129.54" width="0.1524" layer="91"/>
 <junction x="175.26" y="129.54"/>
-</segment>
-</net>
-<net name="!BOOT" class="0">
-<segment>
-<pinref part="R4" gate="G$1" pin="2"/>
-<wire x1="175.26" y1="144.78" x2="175.26" y2="152.4" width="0.1524" layer="91"/>
+<wire x1="175.26" y1="144.78" x2="175.26" y2="147.32" width="0.1524" layer="91"/>
 <label x="175.26" y="152.4" size="1.27" layer="95" font="vector" ratio="20" rot="R90" xref="yes"/>
+<wire x1="175.26" y1="147.32" x2="175.26" y2="152.4" width="0.1524" layer="91"/>
+<wire x1="175.26" y1="129.54" x2="175.26" y2="144.78" width="0.1524" layer="91"/>
 </segment>
 <segment>
@@
 <segment>
 <pinref part="R10" gate="G$1" pin="2"/>
-<pinref part="D2" gate="G$1" pin="C"/>
-<wire x1="116.84" y1="78.74" x2="121.92" y2="78.74" width="0.1524" layer="91"/>
-</segment>
-</net>
+<pinref part="D2" gate="G$1" pin="A"/>
+<wire x1="116.84" y1="78.74" x2="124.46" y2="78.74" width="0.1524" layer="91"/>
+</segment>
+</net>
